Commit message: 3d lidar implemented

File: install/my_tracked_robot_description/share/my_tracked_robot_description/urdf/tracked_robot.urdf.xacro (robot description, xacro)
@@ -1,190 +1,120 @@
 <?xml version="1.0"?>
+<!-- IMPORTANT: The name is kept as "tracked_robot" to match your launch files. -->
 <robot xmlns:xacro="http://www.ros.org/wiki/xacro" name="tracked_robot">
-    <!-- Define Robot constants -->
-    <xacro:property name="chassis_length" value="0.4"/>
+    <!-- #################### PROPERTIES #################### -->
+    <xacro:property name="PI" value="3.1415926535897931"/>
+    <!-- Chassis Properties -->
+    <xacro:property name="chassis_length" value="0.5"/>
     <xacro:property name="chassis_width" value="0.3"/>
     <xacro:property name="chassis_height" value="0.15"/>
     <xacro:property name="chassis_mass" value="5.0"/>
-    <!-- Track properties (for visual and collision) -->
-    <xacro:property name="track_length" value="0.35"/>
-    <xacro:property name="track_width" value="0.06"/>
-    <xacro:property name="track_height" value="0.08"/>
-    <xacro:property name="track_mass" value="1.0"/>
-    <xacro:property name="track_separation" value="0.32"/> <!-- Distance between the two tracks -->
-    <!-- Wheel properties (for the diff_drive plugin physics) -->
-    <xacro:property name="wheel_radius" value="${track_height / 2}"/>
-    <!-- Material Definitions -->
-    <material name="blue">
-        <color rgba="0.2 0.4 0.8 1.0"/>
-    </material>
-    <material name="black">
-        <color rgba="0.1 0.1 0.1 1.0"/>
-    </material>
-    <material name="red">
-        <color rgba="0.8 0.1 0.1 1.0"/>
-    </material>
-    <!-- BASE LINK (Chassis) -->
+    <!-- Wheel Properties -->
+    <xacro:property name="wheel_radius" value="0.1"/>
+    <xacro:property name="wheel_width" value="0.05"/>
+    <xacro:property name="wheel_mass" value="0.5"/>
+    <xacro:property name="wheel_separation" value="0.35"/>
+    <xacro:property name="wheel_x_offset" value="-0.2"/>
+    <xacro:property name="wheel_z_offset" value="-0.05"/>
+    <!-- Caster Properties -->
+    <xacro:property name="caster_radius" value="0.05"/>
+    <xacro:property name="caster_mass" value="0.1"/>
+    <xacro:property name="caster_x_offset" value="0.2"/>
+    <xacro:property name="caster_z_offset" value="-0.1"/>
+    <!-- Lidar Properties -->
+    <xacro:property name="lidar_radius" value="0.1"/>
+    <xacro:property name="lidar_length" value="0.05"/>
+    <xacro:property name="lidar_mass" value="0.2"/>
+    <xacro:property name="lidar_z_offset" value="0.1"/>
+    <!-- #################### ROBOT LINKS AND JOINTS #################### -->
     <link name="base_link">
         <visual>
-            <geometry>
-                <box size="${chassis_length} ${chassis_width} ${chassis_height}"/>
-            </geometry>
-            <material name="blue"/>
+            <geometry><box size="${chassis_length} ${chassis_width} ${chassis_height}"/></geometry>
+            <material name="blue"><color rgba="0 0 0.8 1"/></material>
         </visual>
         <collision>
-            <geometry>
-                <box size="${chassis_length} ${chassis_width} ${chassis_height}"/>
-            </geometry>
+            <geometry><box size="${chassis_length} ${chassis_width} ${chassis_height}"/></geometry>
         </collision>
         <inertial>
-            <origin xyz="0 0 0" rpy="0 0 0"/>
             <mass value="${chassis_mass}"/>
-            <inertia ixx="0.1" ixy="0.0" ixz="0.0" iyy="0.1" iyz="0.0" izz="0.1"/>
+            <inertia ixx="0.1" ixy="0" ixz="0" iyy="0.1" iyz="0" izz="0.1"/>
         </inertial>
     </link>
-    <!-- WHEEL/TRACK LINKS -->
-    <link name="left_track_link">
-        <visual>
-            <geometry>
-                <box size="${track_length} ${track_width} ${track_height}"/>
-            </geometry>
-            <material name="black"/>
-        </visual>
-        <collision>
-            <geometry>
-                <box size="${track_length} ${track_width} ${track_height}"/>
-            </geometry>
-            <!-- NEW: Added friction properties for Gazebo -->
-            <surface>
-                <friction>
-                    <ode>
-                        <mu>1.0</mu>  <!-- Primary friction (forward/backward) -->
-                        <mu2>0.2</mu2> <!-- Secondary friction (sideways) -->
-                    </ode>
-                </friction>
-            </surface>
-        </collision>
+    <xacro:macro name="wheel" params="side side_y_reflect">
+        <link name="${side}_wheel_link">
+            <visual>
+                <origin rpy="${PI/2} 0 0" xyz="0 0 0"/>
+                <geometry><cylinder radius="${wheel_radius}" length="${wheel_width}"/></geometry>
+                <material name="black"><color rgba="0 0 0 1"/></material>
+            </visual>
+            <collision>
+                <origin rpy="${PI/2} 0 0" xyz="0 0 0"/>
+                <geometry><cylinder radius="${wheel_radius}" length="${wheel_width}"/></geometry>
+            </collision>
+            <inertial>
+                <mass value="${wheel_mass}"/>
+                <inertia ixx="0.01" ixy="0" ixz="0" iyy="0.01" iyz="0" izz="0.01"/>
+            </inertial>
+        </link>
+        <joint name="${side}_wheel_joint" type="continuous">
+            <parent link="base_link"/>
+            <child link="${side}_wheel_link"/>
+            <origin rpy="0 0 0" xyz="${wheel_x_offset} ${side_y_reflect * wheel_separation/2} ${wheel_z_offset}"/>
+            <axis xyz="0 1 0"/>
+        </joint>
+    </xacro:macro>
+    <xacro:wheel side="left"  side_y_reflect="1"/>
+    <xacro:wheel side="right" side_y_reflect="-1"/>
+    <link name="caster_wheel_link">
+        <visual><geometry><sphere radius="${caster_radius}"/></geometry><material name="black"><color rgba="0 0 0 1"/></material></visual>
+        <collision><geometry><sphere radius="${caster_radius}"/></geometry></collision>
         <inertial>
-            <mass value="${track_mass}"/>
-            <inertia ixx="0.1" ixy="0.0" ixz="0.0" iyy="0.1" iyz="0.0" izz="0.1"/>
+            <mass value="${caster_mass}"/>
+            <inertia ixx="0.01" ixy="0" ixz="0" iyy="0.01" iyz="0" izz="0.01"/>
         </inertial>
     </link>
-    <link name="right_track_link">
-        <visual>
-            <geometry>
-                <box size="${track_length} ${track_width} ${track_height}"/>
-            </geometry>
-            <material name="black"/>
-        </visual>
-        <collision>
-            <geometry>
-                <box size="${track_length} ${track_width} ${track_height}"/>
-            </geometry>
-            <!-- NEW: Added friction properties for Gazebo -->
-            <surface>
-                <friction>
-                    <ode>
-                        <mu>1.0</mu>
-                        <mu2>0.2</mu2>
-                    </ode>
-                </friction>
-            </surface>
-        </collision>
+    <joint name="caster_wheel_joint" type="fixed"><parent link="base_link"/><child link="caster_wheel_link"/><origin xyz="${caster_x_offset} 0 ${caster_z_offset}"/></joint>
+    <link name="lidar_link">
+        <visual><geometry><cylinder length="${lidar_length}" radius="${lidar_radius}"/></geometry><material name="green"><color rgba="0 1 0 1"/></material></visual>
+        <collision><geometry><cylinder length="${lidar_length}" radius="${lidar_radius}"/></geometry></collision>
         <inertial>
-            <mass value="${track_mass}"/>
-            <inertia ixx="0.1" ixy="0.0" ixz="0.0" iyy="0.1" iyz="0.0" izz="0.1"/>
+            <mass value="${lidar_mass}"/>
+            <inertia ixx="0.001" ixy="0" ixz="0" iyy="0.001" iyz="0" izz="0.001"/>
         </inertial>
     </link>
-    <!-- JOINTS -->
-    <!-- The joints are still 'continuous' like wheels for the plugin -->
-    <joint name="left_track_joint" type="continuous">
-        <parent link="base_link"/>
-        <child link="left_track_link"/>
-        <origin xyz="0 ${track_separation/2} -${chassis_height/2 - track_height/2}" rpy="0 0 0"/>
-        <axis xyz="0 1 0"/>
-    </joint>
-    <joint name="right_track_joint" type="continuous">
-        <parent link="base_link"/>
-        <child link="right_track_link"/>
-        <origin xyz="0 -${track_separation/2} -${chassis_height/2 - track_height/2}" rpy="0 0 0"/>
-        <axis xyz="0 1 0"/>
-    </joint>
-    <!-- SENSORS -->
-    <link name="laser_link">
-        <visual>
-            <geometry>
-                <cylinder radius="0.03" length="0.05"/>
-            </geometry>
-            <material name="red"/> <!-- This will now work -->
-        </visual>
-        <collision>
-            <geometry>
-                <cylinder radius="0.03" length="0.05"/>
-            </geometry>
-        </collision>
-        <inertial>
-            <mass value="0.1"/>
-            <inertia ixx="0.001" ixy="0.0" ixz="0.0" iyy="0.001" iyz="0.0" izz="0.001"/>
-        </inertial>
-    </link>
-    <joint name="laser_joint" type="fixed">
-        <parent link="base_link"/>
-        <child link="laser_link"/>
-        <origin xyz="${chassis_length/2 - 0.025} 0 ${chassis_height/2}" rpy="0 0 0"/>
-    </joint>
-    <!-- GAZEBO PLUGINS -->
+    <joint name="lidar_joint" type="fixed"><parent link="base_link"/><child link="lidar_link"/><origin xyz="0.15 0 ${lidar_z_offset}"/></joint>
+    <!-- #################### GAZEBO PLUGINS AND REFERENCES #################### -->
+    <gazebo reference="base_link"><material>Gazebo/Blue</material></gazebo>
+    <gazebo reference="left_wheel_link"><material>Gazebo/Black</material></gazebo>
+    <gazebo reference="right_wheel_link"><material>Gazebo/Black</material></gazebo>
+    <gazebo reference="lidar_link"><material>Gazebo/Green</material></gazebo>
+    <gazebo reference="caster_wheel_link"><material>Gazebo/Black</material><mu1>0.1</mu1><mu2>0.1</mu2></gazebo>
     <gazebo>
         <plugin name="diff_drive" filename="libgazebo_ros_diff_drive.so">
-            <ros>
-                <namespace>/</namespace>
-            </ros>
-            <!-- UPDATED: Point to the new joint names -->
-            <left_joint>left_track_joint</left_joint>
-            <right_joint>right_track_joint</right_joint>
-            <!-- These are still based on "wheels" for physics calculation -->
-            <wheel_separation>${track_separation}</wheel_separation>
+            <ros><remapping>cmd_vel:=cmd_vel</remapping><remapping>odom:=odom</remapping></ros>
+            <left_joint>left_wheel_joint</left_joint>
+            <right_joint>right_wheel_joint</right_joint>
+            <wheel_separation>${wheel_separation}</wheel_separation>
             <wheel_diameter>${2*wheel_radius}</wheel_diameter>
-            <max_wheel_torque>100</max_wheel_torque> <!-- Increased torque just in case -->
-            <max_wheel_acceleration>10.0</max_wheel_acceleration>
+            <max_wheel_torque>20</max_wheel_torque>
+            <max_wheel_acceleration>1.0</max_wheel_acceleration>
+            <odometry_frame>odom</odometry_frame>
+            <robot_base_frame>base_link</robot_base_frame>
             <publish_odom>true</publish_odom>
             <publish_odom_tf>true</publish_odom_tf>
-            <publish_wheel_tf>false</publish_wheel_tf>
-            <odometry_frame>odom</odometry_frame>
-            <robot_base_frame>base_link</robot_base_frame>
         </plugin>
     </gazebo>
-    <gazebo reference="laser_link">
-        <sensor name="laser" type="ray">
-            <!-- ... (rest of sensor plugin is the same) ... -->
-            <pose>0 0 0 0 0 0</pose>
-            <visualize>true</visualize>
-            <update_rate>10</update_rate>
+    <gazebo reference="lidar_link">
+        <sensor name="lidar_sensor" type="ray">
+            <visualize>true</visualize><update_rate>10</update_rate>
             <ray>
                 <scan>
-                    <horizontal>
-                        <samples>360</samples>
-                        <resolution>1</resolution>
-                        <min_angle>-3.14159</min_angle>
-                        <max_angle>3.14159</max_angle>
-                    </horizontal>
+                    <horizontal><samples>360</samples><min_angle>-${PI}</min_angle><max_angle>${PI}</max_angle></horizontal>
                 </scan>
-                <range>
-                    <min>0.12</min>
-                    <max>10.0</max>
-                    <resolution>0.01</resolution>
-                </range>
-                <noise>
-                    <type>gaussian</type>
-                    <mean>0.0</mean>
-                    <stddev>0.01</stddev>
-                </noise>
+                <range><min>0.14</min><max>2.0</max></range>
             </ray>
-            <plugin name="laser_controller" filename="libgazebo_ros_ray_sensor.so">
-                <ros>
-                    <namespace>/</namespace>
-                    <argument>--ros-args -r ~/out:=scan</argument>
-                </ros>
+            <plugin name="lidar_controller" filename="libgazebo_ros_ray_sensor.so">
+                <ros><remapping>~/out:=scan</remapping></ros>
                 <output_type>sensor_msgs/LaserScan</output_type>
-                <frame_name>laser_link</frame_name>
+                <frame_name>lidar_link</frame_name>
             </plugin>
         </sensor>

File: my_tracked_robot_description/urdf/tracked_robot.urdf.xacro (robot description, xacro)
@@ -21,9 +21,13 @@
     <xacro:property name="caster_x_offset" value="0.2"/>
     <xacro:property name="caster_z_offset" value="-0.1"/>
-    <!-- Lidar Properties -->
-    <xacro:property name="lidar_radius" value="0.1"/>
-    <xacro:property name="lidar_length" value="0.05"/>
-    <xacro:property name="lidar_mass" value="0.2"/>
+    <!-- 2D Lidar Properties (Original) -->
+    <xacro:property name="lidar_2d_radius" value="0.1"/>
+    <xacro:property name="lidar_2d_length" value="0.05"/>
+    <xacro:property name="lidar_2d_mass" value="0.2"/>
     <xacro:property name="lidar_z_offset" value="0.1"/>
+    <!-- SICK multiScan136 3D Lidar Properties (New) -->
+    <xacro:property name="lidar_3d_radius" value="0.05015"/> <!-- 100.3mm diameter / 2 -->
+    <xacro:property name="lidar_3d_length" value="0.0985"/>  <!-- 98.5mm height -->
+    <xacro:property name="lidar_3d_mass" value="0.7"/>       <!-- 0.7 kg -->
     <!-- #################### ROBOT LINKS AND JOINTS #################### -->
     <link name="base_link">
@@ -74,18 +78,30 @@
     </link>
     <joint name="caster_wheel_joint" type="fixed"><parent link="base_link"/><child link="caster_wheel_link"/><origin xyz="${caster_x_offset} 0 ${caster_z_offset}"/></joint>
-    <link name="lidar_link">
-        <visual><geometry><cylinder length="${lidar_length}" radius="${lidar_radius}"/></geometry><material name="green"><color rgba="0 1 0 1"/></material></visual>
-        <collision><geometry><cylinder length="${lidar_length}" radius="${lidar_radius}"/></geometry></collision>
+    <!-- 2D LiDAR Link (Original, Renamed) -->
+    <link name="lidar_2d_link">
+        <visual><geometry><cylinder length="${lidar_2d_length}" radius="${lidar_2d_radius}"/></geometry><material name="green"><color rgba="0 1 0 1"/></material></visual>
+        <!-- COLLISION REMOVED to prevent interference with the co-located 3D LiDAR -->
         <inertial>
-            <mass value="${lidar_mass}"/>
+            <mass value="${lidar_2d_mass}"/>
             <inertia ixx="0.001" ixy="0" ixz="0" iyy="0.001" iyz="0" izz="0.001"/>
         </inertial>
     </link>
-    <joint name="lidar_joint" type="fixed"><parent link="base_link"/><child link="lidar_link"/><origin xyz="0.15 0 ${lidar_z_offset}"/></joint>
+    <joint name="lidar_2d_joint" type="fixed"><parent link="base_link"/><child link="lidar_2d_link"/><origin xyz="0.15 0 ${lidar_z_offset}"/></joint>
+    <!-- 3D LiDAR Link (New) -->
+    <link name="lidar_3d_link">
+        <visual><geometry><cylinder length="${lidar_3d_length}" radius="${lidar_3d_radius}"/></geometry><material name="red"><color rgba="1 0 0 1"/></material></visual>
+        <!-- COLLISION REMOVED to prevent interference with the co-located 2D LiDAR -->
+        <inertial>
+            <mass value="${lidar_3d_mass}"/>
+            <inertia ixx="0.001" ixy="0" ixz="0" iyy="0.001" iyz="0" izz="0.001"/>
+        </inertial>
+    </link>
+    <joint name="lidar_3d_joint" type="fixed"><parent link="base_link"/><child link="lidar_3d_link"/><origin xyz="0.15 0 ${lidar_z_offset}"/></joint>
     <!-- #################### GAZEBO PLUGINS AND REFERENCES #################### -->
     <gazebo reference="base_link"><material>Gazebo/Blue</material></gazebo>
     <gazebo reference="left_wheel_link"><material>Gazebo/Black</material></gazebo>
     <gazebo reference="right_wheel_link"><material>Gazebo/Black</material></gazebo>
-    <gazebo reference="lidar_link"><material>Gazebo/Green</material></gazebo>
+    <gazebo reference="lidar_2d_link"><material>Gazebo/Green</material></gazebo>
+    <gazebo reference="lidar_3d_link"><material>Gazebo/Red</material></gazebo> <!-- Material for new 3D LiDAR -->
     <gazebo reference="caster_wheel_link"><material>Gazebo/Black</material><mu1>0.1</mu1><mu2>0.1</mu2></gazebo>
     <gazebo>
@@ -104,6 +120,7 @@
         </plugin>
     </gazebo>
-    <gazebo reference="lidar_link">
-        <sensor name="lidar_sensor" type="ray">
+    <!-- Gazebo Plugin for 2D LiDAR -->
+    <gazebo reference="lidar_2d_link">
+        <sensor name="lidar_2d_sensor" type="ray">
             <visualize>true</visualize><update_rate>10</update_rate>
             <ray>
@@ -113,8 +130,46 @@
                 <range><min>0.14</min><max>2.0</max></range>
             </ray>
-            <plugin name="lidar_controller" filename="libgazebo_ros_ray_sensor.so">
+            <plugin name="lidar_2d_controller" filename="libgazebo_ros_ray_sensor.so">
                 <ros><remapping>~/out:=scan</remapping></ros>
                 <output_type>sensor_msgs/LaserScan</output_type>
-                <frame_name>lidar_link</frame_name>
+                <frame_name>lidar_2d_link</frame_name>
+            </plugin>
+        </sensor>
+    </gazebo>
+    <!-- Gazebo Plugin for SICK multiScan136 3D LiDAR -->
+    <gazebo reference="lidar_3d_link">
+        <sensor name="lidar_3d_sensor" type="ray">
+            <visualize>true</visualize>
+            <update_rate>20</update_rate>
+            <ray>
+                <scan>
+                    <horizontal>
+                        <samples>720</samples>
+                        <resolution>1</resolution>
+                        <min_angle>-${PI}</min_angle>
+                        <max_angle>${PI}</max_angle>
+                    </horizontal>
+                    <vertical>
+                        <samples>14</samples>
+                        <resolution>1</resolution>
+                        <min_angle>-0.7417</min_angle> <!-- -42.5 degrees -->
+                        <max_angle>0.3927</max_angle>  <!-- 22.5 degrees -->
+                    </vertical>
+                </scan>
+                <range>
+                    <min>0.05</min>
+                    <max>1.0</max>
+                    <resolution>0.01</resolution>
+                </range>
+                <noise>
+                    <type>gaussian</type>
+                    <mean>0.0</mean>
+                    <stddev>0.01</stddev>
+                </noise>
+            </ray>
+            <plugin name="lidar_3d_controller" filename="libgazebo_ros_ray_sensor.so">
+                <ros><remapping>~/out:=points</remapping></ros>
+                <output_type>sensor_msgs/PointCloud2</output_type>
+                <frame_name>lidar_3d_link</frame_name>
             </plugin>
         </sensor>
