Commit message: Working U-turn with env and robot modification

File: my_tracked_robot_description/urdf/tracked_robot.urdf.xacro (robot description, xacro)
@@ -1,20 +1,16 @@
 <?xml version="1.0"?>
 <robot xmlns:xacro="http://www.ros.org/wiki/xacro" name="tracked_robot">
-    <!-- Properties -->
-    <xacro:property name="chassis_length" value="0.4"/>
+    <!-- Robot Properties -->
+    <xacro:property name="chassis_length" value="0.3"/>
     <xacro:property name="chassis_width" value="0.3"/>
-    <xacro:property name="chassis_height" value="0.15"/>
+    <xacro:property name="chassis_height" value="0.1"/>
     <xacro:property name="chassis_mass" value="5.0"/>
-    <xacro:property name="track_visual_length" value="0.35"/>
-    <xacro:property name="track_visual_width" value="0.06"/>
-    <xacro:property name="track_visual_height" value="0.08"/>
-    <xacro:property name="track_separation" value="0.32"/> <!-- Separation between left/right wheel sets -->
-    <!-- Wheel Properties -->
-    <xacro:property name="wheel_radius" value="${track_visual_height / 2}"/>
-    <xacro:property name="wheel_width" value="${track_visual_width * 0.9}"/> <!-- Slightly narrower than track visual -->
+    <xacro:property name="wheel_separation" value="0.3"/>
+    <xacro:property name="wheel_radius" value="0.1"/>
+    <xacro:property name="wheel_width" value="0.1"/>
     <xacro:property name="wheel_mass" value="0.5"/>
-    <xacro:property name="wheel_x_spacing" value="${track_visual_length * 0.7}"/> <!-- Distance between front and rear wheel centers on one side -->
+    <xacro:property name="wheel_x_spacing" value="0.25"/>
     <xacro:property name="PI" value="3.1415926535897931"/>
-    <!-- Inertial calculation macro for a box -->
+    <!-- Inertial Macros -->
     <xacro:macro name="inertial_box" params="mass x y z">
         <inertial>
@@ -25,5 +21,4 @@
         </inertial>
     </xacro:macro>
-    <!-- Inertial calculation macro for a cylinder aligned along Y (for wheels) -->
     <xacro:macro name="inertial_cylinder_y" params="mass radius length">
       <inertial>
@@ -34,7 +29,6 @@
       </inertial>
     </xacro:macro>
-    <!-- Base Footprint (Dummy Link) -->
+    <!-- Robot Links and Joints -->
     <link name="base_footprint"/>
-    <!-- Base Link (Chassis) -->
     <link name="base_link">
         <visual>
@@ -47,4 +41,7 @@
         <xacro:inertial_box mass="${chassis_mass}" x="${chassis_length}" y="${chassis_width}" z="${chassis_height}"/>
     </link>
+    <gazebo reference="base_link">
+        <material>Gazebo/Purple</material>
+    </gazebo>
     <joint name="base_footprint_joint" type="fixed">
         <parent link="base_footprint"/>
@@ -52,5 +49,4 @@
         <origin xyz="0 0 ${chassis_height/2 + wheel_radius}" rpy="0 0 0"/>
     </joint>
-    <!-- WHEEL MACRO -->
     <xacro:macro name="wheel" params="prefix side side_y_reflect x_offset">
         <link name="${prefix}_${side}_wheel_link">
@@ -58,5 +54,5 @@
                 <origin xyz="0 0 0" rpy="${PI/2} 0 0"/>
                 <geometry><cylinder radius="${wheel_radius}" length="${wheel_width}"/></geometry>
-                <material name="${side}_wheel_color"><color rgba="0.2 0.2 0.2 1"/></material>
+                <material name="wheel_grey"><color rgba="0.2 0.2 0.2 1"/></material>
             </visual>
             <collision>
@@ -69,45 +65,23 @@
             <parent link="base_link"/>
             <child link="${prefix}_${side}_wheel_link"/>
-            <origin xyz="${x_offset} ${side_y_reflect * track_separation/2} -${chassis_height/2}" rpy="0 0 0"/>
+            <origin xyz="${x_offset} ${side_y_reflect * wheel_separation/2} -${chassis_height/2}" rpy="0 0 0"/>
             <axis xyz="0 1 0"/>
         </joint>
         <gazebo reference="${prefix}_${side}_wheel_link">
-          <material>Gazebo/DarkGrey</material>
-          <mu1>1.0</mu1>
-          <mu2>0.1</mu2>
-          <kp>500000.0</kp>
-          <kd>10.0</kd>
-          <implicitSpringDamper>1</implicitSpringDamper>
-          <minDepth>0.001</minDepth>
+            <material>Gazebo/DarkGrey</material>
+            <xacro:if value="${prefix == 'rear'}">
+                <mu1>100.0</mu1>
+                <mu2>1.0</mu2>
+            </xacro:if>
+            <xacro:if value="${prefix == 'front'}">
+                <mu1>100.0</mu1>
+                <mu2>1.0</mu2>
+            </xacro:if>
         </gazebo>
     </xacro:macro>
-    <!-- Instantiate Wheels -->
     <xacro:wheel prefix="front" side="left"  side_y_reflect="1"  x_offset="${wheel_x_spacing/2}"/>
     <xacro:wheel prefix="rear"  side="left"  side_y_reflect="1"  x_offset="-${wheel_x_spacing/2}"/>
     <xacro:wheel prefix="front" side="right" side_y_reflect="-1" x_offset="${wheel_x_spacing/2}"/>
     <xacro:wheel prefix="rear"  side="right" side_y_reflect="-1" x_offset="-${wheel_x_spacing/2}"/>
-    <!-- Track Visual Links -->
-    <link name="left_track_visual_link">
-        <visual>
-            <geometry><box size="${track_visual_length} ${track_visual_width} ${track_visual_height}"/></geometry>
-            <material name="track_orange_material"><color rgba="1.0 0.5 0.0 1.0"/></material>
-        </visual>
-    </link>
-    <link name="right_track_visual_link">
-        <visual>
-            <geometry><box size="${track_visual_length} ${track_visual_width} ${track_visual_height}"/></geometry>
-            <material name="track_orange_material"/>
-        </visual>
-    </link>
-    <joint name="left_track_visual_joint" type="fixed">
-        <parent link="base_link"/>
-        <child link="left_track_visual_link"/>
-        <origin xyz="0 ${track_separation/2} -${chassis_height/2}" rpy="0 0 0"/>
-    </joint>
-    <joint name="right_track_visual_joint" type="fixed">
-        <parent link="base_link"/>
-        <child link="right_track_visual_link"/>
-        <origin xyz="0 -${track_separation/2} -${chassis_height/2}" rpy="0 0 0"/>
-    </joint>
     <!-- Lidar Sensor -->
     <link name="laser_link">
@@ -119,75 +93,69 @@
         <parent link="base_link"/>
         <child link="laser_link"/>
-        <origin xyz="${chassis_length/2 - 0.025} 0 ${chassis_height/2 + 0.025 + 0.01}" rpy="0 0 0"/>
+        <origin xyz="${chassis_length/2 - 0.025} 0 ${chassis_height/2 + 0.05}" rpy="0 0 0"/>
     </joint>
-    <!-- GAZEBO Material TAGS -->
-    <gazebo reference="base_link"><material>Gazebo/Purple</material></gazebo>
-    <gazebo reference="left_track_visual_link"><material>Gazebo/Orange</material></gazebo>
-    <gazebo reference="right_track_visual_link"><material>Gazebo/Orange</material></gazebo>
-    <gazebo reference="laser_link"><material>Gazebo/Red</material></gazebo>
-    <!-- Gazebo Plugins -->
+<!-- Gazebo Plugins -->
     <gazebo>
-        <plugin name="diff_drive" filename="libgazebo_ros_diff_drive.so">
-            <ros></ros> <!-- Ensuring empty tag as per original -->
+        <!-- Plugin for the REAR wheels -->
+        <plugin name="diff_drive_rear" filename="libgazebo_ros_diff_drive.so">
+            <ros>
+                <remapping>cmd_vel:=/cmd_vel</remapping>
+                <remapping>odom:=/odom</remapping> <!-- This plugin will publish odometry -->
+            </ros>
+            <!-- Rear wheels -->
             <left_joint>rear_left_wheel_joint</left_joint>
             <right_joint>rear_right_wheel_joint</right_joint>
-            <wheel_separation>${track_separation}</wheel_separation>
+            <wheel_separation>${wheel_separation}</wheel_separation>
             <wheel_diameter>${2*wheel_radius}</wheel_diameter>
             <max_wheel_torque>200</max_wheel_torque>
-            <max_wheel_acceleration>20.0</max_wheel_acceleration>
+            <max_wheel_acceleration>5.0</max_wheel_acceleration>
+            <!-- Odometry configuration -->
+            <odometry_frame>odom</odometry_frame>
+            <robot_base_frame>base_footprint</robot_base_frame>
             <publish_odom>true</publish_odom>
             <publish_odom_tf>true</publish_odom_tf>
-            <publish_wheel_tf>false</publish_wheel_tf>
-            <publish_wheel_joint_state>true</publish_wheel_joint_state>
-            <odometry_frame>odom</odometry_frame>
-            <robot_base_frame>base_footprint</robot_base_frame>
-            <update_rate>50</update_rate>
+        </plugin>
+        <!-- Plugin for the FRONT wheels -->
+        <plugin name="diff_drive_front" filename="libgazebo_ros_diff_drive.so">
+            <ros>
+                <remapping>cmd_vel:=/cmd_vel</remapping>
+            </ros>
+            <!-- Front wheels -->
+            <left_joint>front_left_wheel_joint</left_joint>
+            <right_joint>front_right_wheel_joint</right_joint>
+            <wheel_separation>${wheel_separation}</wheel_separation>
+            <wheel_diameter>${2*wheel_radius}</wheel_diameter>
+            <max_wheel_torque>200</max_wheel_torque>
+            <max_wheel_acceleration>5.0</max_wheel_acceleration>
+            <!-- Disable odometry from this plugin to avoid conflicts -->
+            <publish_odom>false</publish_odom>
+            <publish_odom_tf>false</publish_odom_tf>
         </plugin>
     </gazebo>
-    <!-- In your current tracked_robot.xacro -->
     <gazebo reference="laser_link">
+        <material>Gazebo/Red</material>
         <sensor name="laser" type="ray">
             <visualize>true</visualize>
             <update_rate>10</update_rate>
             <ray>
-                <scan><horizontal><samples>360</samples><min_angle>-${PI}</min_angle><max_angle>${PI}</max_angle></horizontal></scan>
+                <scan>
+                    <horizontal>
+                        <samples>360</samples>
+                        <min_angle>-${PI}</min_angle>
+                        <max_angle>${PI}</max_angle>
+                    </horizontal>
+                </scan>
                 <range>
-                    <min>0.12</min>
-                    <max>2.0</max> <!-- KEEP THIS CHANGE for 2m range -->
-                    <resolution>0.015</resolution>
+                    <min>0.14</min>
+                    <max>2.0</max>
                 </range>
-                <noise><type>gaussian</type><mean>0.0</mean><stddev>0.01</stddev></noise>
             </ray>
             <plugin name="laser_controller" filename="libgazebo_ros_ray_sensor.so">
                 <ros>
-                    <namespace>/laser_controller</namespace> <!-- KEEP NAMESPACE -->
-                    <remapping>~/out:=out</remapping>    <!-- KEEP REMAPPING (topic becomes /laser_controller/out) -->
+                    <namespace>/laser_controller</namespace>
+                    <remapping>~/out:=scan</remapping>
                 </ros>
                 <output_type>sensor_msgs/LaserScan</output_type>
                 <frame_name>laser_link</frame_name>
-                <!-- topic_name is not needed when using namespace + remapping for this specific outcome -->
-            </plugin>
-        </sensor>
-    </gazebo>
-   <!-- ========= GAZEBO-SPECIFIC PROPERTIES FOR THE ROBOT BODY ======== -->
-    <!-- ====================================================================== -->
-    <!-- ====================================================================== -->
-    <gazebo reference="base_link">
-        <!-- 1. Set the visual material -->
-        <material>Gazebo/Purple</material>
-        <!-- 2. Attach the Bumper/Contact Sensor -->
-        <sensor name="contact_sensor" type="contact">
-            <always_on>true</always_on>
-            <update_rate>50.0</update_rate>
-            <contact>
-                <!-- This MUST match the name in the base_link's collision tag -->
-                <collision>base_link_collision</collision>
-            </contact>
-            <plugin name="gazebo_ros_bumper" filename="libgazebo_ros_bumper.so">
-                <ros>
-                    <!-- Remap the output topic for clarity -->
-                    <remapping>~/out:=bumper_states</remapping>
-                </ros>
-                <frame_name>base_link</frame_name>
             </plugin>
         </sensor>
