Commit message: working urdf with simulation modification to remove bumbness road

File: my_tracked_robot_description/urdf/tracked_robot.urdf.xacro (robot description, xacro)
@@ -1,161 +1,127 @@
 <?xml version="1.0"?>
+<!-- IMPORTANT: The name is kept as "tracked_robot" to match your launch files. -->
 <robot xmlns:xacro="http://www.ros.org/wiki/xacro" name="tracked_robot">
-    <!-- Robot Properties -->
-    <xacro:property name="chassis_length" value="0.3"/>
+    <!-- #################### PROPERTIES #################### -->
+    <xacro:property name="PI" value="3.1415926535897931"/>
+    <!-- Chassis Properties -->
+    <xacro:property name="chassis_length" value="0.5"/>
     <xacro:property name="chassis_width" value="0.3"/>
-    <xacro:property name="chassis_height" value="0.1"/>
+    <xacro:property name="chassis_height" value="0.15"/>
     <xacro:property name="chassis_mass" value="5.0"/>
-    <xacro:property name="wheel_separation" value="0.3"/>
+    <!-- Wheel Properties -->
     <xacro:property name="wheel_radius" value="0.1"/>
-    <xacro:property name="wheel_width" value="0.1"/>
+    <xacro:property name="wheel_width" value="0.05"/>
     <xacro:property name="wheel_mass" value="0.5"/>
-    <xacro:property name="wheel_x_spacing" value="0.25"/>
-    <xacro:property name="PI" value="3.1415926535897931"/>
-    <!-- Inertial Macros -->
-    <xacro:macro name="inertial_box" params="mass x y z">
-        <inertial>
-            <mass value="${mass}"/>
-            <inertia ixx="${(1/12) * mass * (y*y + z*z)}" ixy="0.0" ixz="0.0"
-                     iyy="${(1/12) * mass * (x*x + z*z)}" iyz="0.0"
-                     izz="${(1/12) * mass * (x*x + y*y)}"/>
-        </inertial>
-    </xacro:macro>
-    <xacro:macro name="inertial_cylinder_y" params="mass radius length">
-      <inertial>
-        <mass value="${mass}"/>
-        <inertia ixx="${(1/12)*mass*(3*radius*radius + length*length)}" ixy="0.0" ixz="0.0"
-                 iyy="${(1/2)*mass*radius*radius}" iyz="0.0"
-                 izz="${(1/12)*mass*(3*radius*radius + length*length)}"/>
-      </inertial>
-    </xacro:macro>
-    <!-- Robot Links and Joints -->
-    <link name="base_footprint"/>
+    <xacro:property name="wheel_separation" value="0.35"/>
+    <xacro:property name="wheel_x_offset" value="-0.2"/>
+    <xacro:property name="wheel_z_offset" value="-0.05"/>
+    <!-- Caster Properties -->
+    <xacro:property name="caster_radius" value="0.05"/>
+    <xacro:property name="caster_mass" value="0.1"/>
+    <xacro:property name="caster_x_offset" value="0.2"/>
+    <xacro:property name="caster_z_offset" value="-0.1"/>
+    <!-- Lidar Properties -->
+    <xacro:property name="lidar_radius" value="0.1"/>
+    <xacro:property name="lidar_length" value="0.05"/>
+    <xacro:property name="lidar_mass" value="0.2"/>
+    <xacro:property name="lidar_z_offset" value="0.1"/>
+    <!-- #################### ROBOT LINKS AND JOINTS #################### -->
     <link name="base_link">
         <visual>
             <geometry><box size="${chassis_length} ${chassis_width} ${chassis_height}"/></geometry>
-            <material name="chassis_purple"><color rgba="0.5 0.0 0.5 1.0"/></material>
+            <material name="blue"><color rgba="0 0 0.8 1"/></material>
         </visual>
-        <collision name="base_link_collision">
+        <collision>
             <geometry><box size="${chassis_length} ${chassis_width} ${chassis_height}"/></geometry>
         </collision>
-        <xacro:inertial_box mass="${chassis_mass}" x="${chassis_length}" y="${chassis_width}" z="${chassis_height}"/>
+        <inertial>
+            <mass value="${chassis_mass}"/>
+            <inertia ixx="0.1" ixy="0" ixz="0" iyy="0.1" iyz="0" izz="0.1"/>
+        </inertial>
     </link>
-    <gazebo reference="base_link">
-        <material>Gazebo/Purple</material>
-    </gazebo>
-    <joint name="base_footprint_joint" type="fixed">
-        <parent link="base_footprint"/>
-        <child link="base_link"/>
-        <origin xyz="0 0 ${chassis_height/2 + wheel_radius}" rpy="0 0 0"/>
-    </joint>
-    <xacro:macro name="wheel" params="prefix side side_y_reflect x_offset">
-        <link name="${prefix}_${side}_wheel_link">
+    <xacro:macro name="wheel" params="side side_y_reflect">
+        <link name="${side}_wheel_link">
             <visual>
-                <origin xyz="0 0 0" rpy="${PI/2} 0 0"/>
+                <origin rpy="${PI/2} 0 0" xyz="0 0 0"/>
                 <geometry><cylinder radius="${wheel_radius}" length="${wheel_width}"/></geometry>
-                <material name="wheel_grey"><color rgba="0.2 0.2 0.2 1"/></material>
+                <material name="black"><color rgba="0 0 0 1"/></material>
             </visual>
             <collision>
-                <origin xyz="0 0 0" rpy="${PI/2} 0 0"/>
+                <origin rpy="${PI/2} 0 0" xyz="0 0 0"/>
                 <geometry><cylinder radius="${wheel_radius}" length="${wheel_width}"/></geometry>
             </collision>
-            <xacro:inertial_cylinder_y mass="${wheel_mass}" radius="${wheel_radius}" length="${wheel_width}"/>
+            <inertial>
+                <mass value="${wheel_mass}"/>
+                <inertia ixx="0.01" ixy="0" ixz="0" iyy="0.01" iyz="0" izz="0.01"/>
+            </inertial>
         </link>
-        <joint name="${prefix}_${side}_wheel_joint" type="continuous">
+        <joint name="${side}_wheel_joint" type="continuous">
             <parent link="base_link"/>
-            <child link="${prefix}_${side}_wheel_link"/>
-            <origin xyz="${x_offset} ${side_y_reflect * wheel_separation/2} -${chassis_height/2}" rpy="0 0 0"/>
+            <child link="${side}_wheel_link"/>
+            <origin rpy="0 0 0" xyz="${wheel_x_offset} ${side_y_reflect * wheel_separation/2} ${wheel_z_offset}"/>
             <axis xyz="0 1 0"/>
         </joint>
-        <gazebo reference="${prefix}_${side}_wheel_link">
-            <material>Gazebo/DarkGrey</material>
-            <xacro:if value="${prefix == 'rear'}">
-                <mu1>100.0</mu1>
-                <mu2>1.0</mu2>
-            </xacro:if>
-            <xacro:if value="${prefix == 'front'}">
-                <mu1>100.0</mu1>
-                <mu2>1.0</mu2>
-            </xacro:if>
-        </gazebo>
     </xacro:macro>
-    <xacro:wheel prefix="front" side="left"  side_y_reflect="1"  x_offset="${wheel_x_spacing/2}"/>
-    <xacro:wheel prefix="rear"  side="left"  side_y_reflect="1"  x_offset="-${wheel_x_spacing/2}"/>
-    <xacro:wheel prefix="front" side="right" side_y_reflect="-1" x_offset="${wheel_x_spacing/2}"/>
-    <xacro:wheel prefix="rear"  side="right" side_y_reflect="-1" x_offset="-${wheel_x_spacing/2}"/>
-    <!-- Lidar Sensor -->
-    <link name="laser_link">
-        <visual><geometry><cylinder radius="0.03" length="0.05"/></geometry></visual>
-        <collision><geometry><cylinder radius="0.03" length="0.05"/></geometry></collision>
-        <xacro:inertial_box mass="0.1" x="0.06" y="0.06" z="0.05"/>
+    <xacro:wheel side="left"  side_y_reflect="1"/>
+    <xacro:wheel side="right" side_y_reflect="-1"/>
+    <link name="caster_wheel_link">
+        <visual><geometry><sphere radius="${caster_radius}"/></geometry><material name="black"><color rgba="0 0 0 1"/></material></visual>
+        <collision><geometry><sphere radius="${caster_radius}"/></geometry></collision>
+        <inertial>
+            <mass value="${caster_mass}"/>
+            <inertia ixx="0.01" ixy="0" ixz="0" iyy="0.01" iyz="0" izz="0.01"/>
+        </inertial>
     </link>
-    <joint name="laser_joint" type="fixed">
-        <parent link="base_link"/>
-        <child link="laser_link"/>
-        <origin xyz="${chassis_length/2 - 0.025} 0 ${chassis_height/2 + 0.05}" rpy="0 0 0"/>
-    </joint>
-<!-- Gazebo Plugins -->
+    <joint name="caster_wheel_joint" type="fixed"><parent link="base_link"/><child link="caster_wheel_link"/><origin xyz="${caster_x_offset} 0 ${caster_z_offset}"/></joint>
+    <link name="lidar_link">
+        <visual><geometry><cylinder length="${lidar_length}" radius="${lidar_radius}"/></geometry><material name="green"><color rgba="0 1 0 1"/></material></visual>
+        <collision><geometry><cylinder length="${lidar_length}" radius="${lidar_radius}"/></geometry></collision>
+        <inertial>
+            <mass value="${lidar_mass}"/>
+            <inertia ixx="0.001" ixy="0" ixz="0" iyy="0.001" iyz="0" izz="0.001"/>
+        </inertial>
+    </link>
+    <joint name="lidar_joint" type="fixed"><parent link="base_link"/><child link="lidar_link"/><origin xyz="0.15 0 ${lidar_z_offset}"/></joint>
+    <!-- #################### GAZEBO PLUGINS AND REFERENCES #################### -->
+    <gazebo reference="base_link"><material>Gazebo/Blue</material></gazebo>
+    <gazebo reference="left_wheel_link"><material>Gazebo/Black</material></gazebo>
+    <gazebo reference="right_wheel_link"><material>Gazebo/Black</material></gazebo>
+    <gazebo reference="lidar_link"><material>Gazebo/Green</material></gazebo>
+    <gazebo reference="caster_wheel_link"><material>Gazebo/Black</material><mu1>0.1</mu1><mu2>0.1</mu2></gazebo>
     <gazebo>
-        <!-- Plugin for the REAR wheels -->
-        <plugin name="diff_drive_rear" filename="libgazebo_ros_diff_drive.so">
-            <ros>
-                <remapping>cmd_vel:=/cmd_vel</remapping>
-                <remapping>odom:=/odom</remapping> <!-- This plugin will publish odometry -->
-            </ros>
-            <!-- Rear wheels -->
-            <left_joint>rear_left_wheel_joint</left_joint>
-            <right_joint>rear_right_wheel_joint</right_joint>
+        <plugin name="diff_drive" filename="libgazebo_ros_diff_drive.so">
+            <ros><remapping>cmd_vel:=cmd_vel</remapping><remapping>odom:=odom</remapping></ros>
+            <left_joint>left_wheel_joint</left_joint>
+            <right_joint>right_wheel_joint</right_joint>
             <wheel_separation>${wheel_separation}</wheel_separation>
             <wheel_diameter>${2*wheel_radius}</wheel_diameter>
-            <max_wheel_torque>200</max_wheel_torque>
-            <max_wheel_acceleration>5.0</max_wheel_acceleration>
-            <!-- Odometry configuration -->
+            <max_wheel_torque>20</max_wheel_torque>
+            <max_wheel_acceleration>1.0</max_wheel_acceleration>
             <odometry_frame>odom</odometry_frame>
-            <robot_base_frame>base_footprint</robot_base_frame>
+            <robot_base_frame>base_link</robot_base_frame>
             <publish_odom>true</publish_odom>
             <publish_odom_tf>true</publish_odom_tf>
         </plugin>
-        <!-- Plugin for the FRONT wheels -->
-        <plugin name="diff_drive_front" filename="libgazebo_ros_diff_drive.so">
-            <ros>
-                <remapping>cmd_vel:=/cmd_vel</remapping>
-            </ros>
-            <!-- Front wheels -->
-            <left_joint>front_left_wheel_joint</left_joint>
-            <right_joint>front_right_wheel_joint</right_joint>
-            <wheel_separation>${wheel_separation}</wheel_separation>
-            <wheel_diameter>${2*wheel_radius}</wheel_diameter>
-            <max_wheel_torque>200</max_wheel_torque>
-            <max_wheel_acceleration>5.0</max_wheel_acceleration>
-            <!-- Disable odometry from this plugin to avoid conflicts -->
-            <publish_odom>false</publish_odom>
-            <publish_odom_tf>false</publish_odom_tf>
+        <plugin name="joint_state_publisher" filename="libgazebo_ros_joint_state_publisher.so">
+            <ros><remapping>~/out:=joint_states</remapping></ros>
+            <update_rate>30</update_rate>
+            <joint_name>left_wheel_joint</joint_name>
+            <joint_name>right_wheel_joint</joint_name>
         </plugin>
     </gazebo>
-    <gazebo reference="laser_link">
-        <material>Gazebo/Red</material>
-        <sensor name="laser" type="ray">
-            <visualize>true</visualize>
-            <update_rate>10</update_rate>
+    <gazebo reference="lidar_link">
+        <sensor name="lidar_sensor" type="ray">
+            <visualize>true</visualize><update_rate>10</update_rate>
             <ray>
                 <scan>
-                    <horizontal>
-                        <samples>360</samples>
-                        <min_angle>-${PI}</min_angle>
-                        <max_angle>${PI}</max_angle>
-                    </horizontal>
+                    <horizontal><samples>360</samples><resolution>1</resolution><min_angle>-${PI}</min_angle><max_angle>${PI}</max_angle></horizontal>
                 </scan>
-                <range>
-                    <min>0.14</min>
-                    <max>2.0</max>
-                </range>
+                <range><min>0.15</min><max>2.0</max><resolution>0.01</resolution></range>
+                <noise><type>gaussian</type><mean>0.0</mean><stddev>0.01</stddev></noise>
             </ray>
-            <plugin name="laser_controller" filename="libgazebo_ros_ray_sensor.so">
-                <ros>
-                    <namespace>/laser_controller</namespace>
-                    <remapping>~/out:=scan</remapping>
-                </ros>
+            <plugin name="lidar_controller" filename="libgazebo_ros_ray_sensor.so">
+                <ros><remapping>~/out:=scan</remapping></ros>
                 <output_type>sensor_msgs/LaserScan</output_type>
-                <frame_name>laser_link</frame_name>
+                <frame_name>lidar_link</frame_name>
             </plugin>
         </sensor>

Commit message: general fixes and improvments

File: my_tracked_robot_description/urdf/tracked_robot.urdf.xacro (robot description, xacro)
@@ -39,4 +39,12 @@
     <xacro:property name="camera_z_offset" value="0.1"/>
     <!-- #################### ROBOT LINKS AND JOINTS #################### -->
+    <!-- NEW: This is the new root link at the front edge of the robot. -->
+<!-- It has no visual or collision properties because it's just a reference frame. -->
+    <link name="base_footprint"/>
+    <joint name="base_link_joint" type="fixed">
+    <parent link="base_footprint"/>
+    <child link="base_link"/>
+    <origin xyz="-${chassis_length / 2.0} 0 0" rpy="0 0 0"/>
+    </joint>
     <link name="base_link">
         <visual>
@@ -139,5 +147,5 @@
             <max_wheel_acceleration>1.0</max_wheel_acceleration>
             <odometry_frame>odom</odometry_frame>
-            <robot_base_frame>base_link</robot_base_frame>
+            <robot_base_frame>base_footprint</robot_base_frame>
             <publish_odom>true</publish_odom>
             <publish_odom_tf>true</publish_odom_tf>
@@ -147,5 +155,5 @@
     <gazebo reference="lidar_2d_link">
         <sensor name="lidar_2d_sensor" type="ray">
-            <visualize>true</visualize><update_rate>10</update_rate>
+            <visualize>false</visualize><update_rate>10</update_rate>
             <ray>
                 <scan>
@@ -171,6 +179,6 @@
                         <samples>720</samples>
                         <resolution>1</resolution>
-                        <min_angle>-${2.00}</min_angle>
-                        <max_angle>${2.00}</max_angle>
+                        <min_angle>-${2.0}</min_angle>
+                        <max_angle>${2.0}</max_angle>
                     </horizontal>
                     <vertical>

Commit message: general fixes

File: my_tracked_robot_description/urdf/tracked_robot.urdf.xacro (robot description, xacro)
@@ -13,5 +13,5 @@
     <xacro:property name="wheel_width" value="0.05"/>
     <xacro:property name="wheel_mass" value="0.5"/>
-    <xacro:property name="wheel_separation" value="0.35"/>
+    <xacro:property name="wheel_separation" value="0.25"/>
     <xacro:property name="wheel_x_offset" value="-0.2"/>
     <xacro:property name="wheel_z_offset" value="-0.05"/>

Commit message: rear camera implementation

File: my_tracked_robot_description/urdf/tracked_robot.urdf.xacro (robot description, xacro)
@@ -130,4 +130,23 @@
         <origin xyz="${camera_x_offset} ${camera_y_offset} ${camera_z_offset}" rpy="0 0 0"/>
     </joint>
+        <!-- ########### NEW: REAR CAMERA ########### -->
+    <!-- RGB Camera Link (Rear) -->
+    <link name="camera_rear_link">
+        <visual>
+            <geometry><box size="${camera_width} ${camera_height} ${camera_depth}"/></geometry>
+            <material name="grey"><color rgba="0.5 0.5 0.5 1"/></material>
+        </visual>
+        <inertial>
+            <mass value="${camera_mass}"/>
+            <inertia ixx="1e-6" ixy="0" ixz="0" iyy="1e-6" iyz="0" izz="1e-6"/>
+        </inertial>
+    </link>
+    <joint name="camera_rear_joint" type="fixed">
+        <parent link="base_link"/>
+        <child link="camera_rear_link"/>
+        <!-- Positioned at the back (-x) and rotated 180 deg (PI rad) around Z to face backward -->
+        <origin xyz="-0.2 ${camera_y_offset} ${camera_z_offset}" rpy="0 0 ${PI}"/>
+    </joint>
+    <!-- ########################################## -->
     <!-- #################### GAZEBO PLUGINS AND REFERENCES #################### -->
     <gazebo reference="base_link"><material>Gazebo/Blue</material></gazebo>
@@ -235,3 +254,35 @@
         </sensor>
     </gazebo>
+        <!-- ########### NEW: GAZEBO PLUGIN FOR REAR CAMERA ########### -->
+    <gazebo reference="camera_rear_link">
+        <material>Gazebo/Grey</material>
+        <sensor type="camera" name="rgb_camera_rear">
+            <update_rate>30.0</update_rate>
+            <camera name="rear_head">
+                <!-- 100 degrees in radians = 1.7453 -->
+                <horizontal_fov>1.7453</horizontal_fov>
+                <image>
+                    <width>1024</width>
+                    <height>576</height>
+                    <format>R8G8B8</format>
+                </image>
+                <clip>
+                    <near>0.28</near>
+                    <far>16.0</far>
+                </clip>
+            </camera>
+            <plugin name="camera_rear_controller" filename="libgazebo_ros_camera.so">
+                <ros>
+                    <namespace>/tracked_robot</namespace>
+                    <remapping>image_raw:=image_raw</remapping>
+                    <remapping>camera_info:=camera_info</remapping>
+                </ros>
+                <!-- This unique camera_name ensures a unique topic: /tracked_robot/rear_camera/image_raw -->
+                <camera_name>rear_camera</camera_name>
+                <frame_name>camera_rear_link</frame_name>
+                <hack_baseline>0.07</hack_baseline>
+            </plugin>
+        </sensor>
+    </gazebo>
+    <!-- ########################################################## -->
 </robot>

Commit message: dynamic mapper size creation, different param for filtering outlier, more work should be done

File: my_tracked_robot_description/urdf/tracked_robot.urdf.xacro (robot description, xacro)
@@ -52,7 +52,7 @@
             <material name="blue"><color rgba="0 0 0.8 1"/></material>
         </visual>
-        <collision>
+        <!-- <collision>
             <geometry><box size="${chassis_length} ${chassis_width} ${chassis_height}"/></geometry>
-        </collision>
+        </collision> -->
         <inertial>
             <mass value="${chassis_mass}"/>

Commit message: feat: implement stratified subset creation for validation dataset; update MC Dropout testing

File: my_tracked_robot_description/urdf/tracked_robot.urdf.xacro (robot description, xacro)
@@ -52,7 +52,7 @@
             <material name="blue"><color rgba="0 0 0.8 1"/></material>
         </visual>
-        <!-- <collision>
+        <collision>
             <geometry><box size="${chassis_length} ${chassis_width} ${chassis_height}"/></geometry>
-        </collision> -->
+        </collision>
         <inertial>
             <mass value="${chassis_mass}"/>
